File: PowerBUS7.brd (EAGLE design)
At the start: 396.2 x 30 mm, 30 parts, among them J1 PIN2F061.040, J2 PIN2F061.040, J3 PIN2F061.040, J4 PIN2F061.040, J5 PIN2F061.040, J6 PIN2F061.040, J7 PIN2F061.040, J8 PIN2F061.040, X1 057-016-1, X10 057-016-1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

Commit message: Add files via upload
Parts:
- moved R2 1.30 mm to (380.5, 16.5), turned to 270 degrees
- moved LED3 1.27 mm to (385.6, 16.5)
- moved J4 1.27 mm to (6.35, 7.11)
- moved J8 1.27 mm to (372.1, 7.11)
- moved J1 1.27 mm to (6.35, 25.4)
- moved J2 1.27 mm to (6.35, 19.1)
- moved J3 1.27 mm to (6.35, 12.7)
- moved J5 1.27 mm to (372.1, 25.4)
- moved J6 1.27 mm to (372.1, 19.1)
- moved J7 1.27 mm to (372.1, 12.7)
- moved JP1 1.27 mm to (135.3, 23.9)
- moved JP2 1.27 mm to (265.0, 23.9)
- moved LED1 1.27 mm to (385.6, 25.4)
- moved LED2 1.27 mm to (385.6, 6.35)
- moved R1 1.27 mm to (380.5, 25.4)
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Routing:
- net 0V: track 49.4 -> 15.8 mm
- net +12V: track 377.8 -> 381.7 mm
- net N$6: track 6.91 -> 5.61 mm
Other:
- board size 396.2 x 30 mm -> 396.2 x 35.1 mm
- board text added: "GATE CV +5V +12V GND GND GND -12V"
- board text added: "RED STRIPE!"
- board text removed: "C:/Users/rage/Desktop/dngr logo inverted.bmp"
- board text removed: "C:/Users/rage/Desktop/dngr text DNGR2.bmp"
- board text removed: "C:/Users/rage/Desktop/dngr text TECH.bmp"
