File: PowerBUS9.brd (EAGLE design)
At the start: 379.4 x 43 mm, 38 parts, among them J1 PIN2F061.040, J2 PIN2F061.040, J3 PIN2F061.040, J4 PIN2F061.040, J5 PIN2F061.040, J6 PIN2F061.040, J7 PIN2F061.040, J8 PIN2F061.040, X1 057-016-1, X10 057-016-1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

Commit message: Add files via upload
Parts:
- moved JP5 1.27 mm to (134.9, 29.1)
Changed lines of the file:
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@@
 <attribute name="NAME" x="333.875165625" y="24.630165625" size="1.27" layer="25" ratio="10"/>
 </element>
-<element name="JP5" library="jumper" package="JP2Q" value="" x="133.628165625" y="29.1084" smashed="yes" rot="R180">
-<attribute name="VALUE" x="129.183165625" y="31.6484" size="1.27" layer="27" ratio="10" rot="R270"/>
+<element name="JP5" library="jumper" package="JP2Q" value="" x="134.898165625" y="29.1084" smashed="yes" rot="R180">
+<attribute name="VALUE" x="130.453165625" y="31.6484" size="1.27" layer="27" ratio="10" rot="R270"/>
 </element>
 <element name="JP1" library="jumper" package="JP2Q" value="" x="235.585" y="29.21" rot="R180"/>
@@
 <wire x1="271.61" y1="30.24" x2="294.17" y2="30.24" width="1.016" layer="16"/>
 <wire x1="171.21" y1="30.24" x2="193.77" y2="30.24" width="1.016" layer="16"/>
-<wire x1="121.01" y1="30.24" x2="132.358165625" y2="30.24" width="1.016" layer="16"/>
-<wire x1="132.358165625" y1="30.24" x2="132.358165625" y2="30.3784" width="1.016" layer="16"/>
-<wire x1="143.57" y1="30.24" x2="134.898165625" y2="30.24" width="1.016" layer="16"/>
-<wire x1="134.898165625" y1="30.24" x2="134.898165625" y2="30.3784" width="1.016" layer="16"/>
 <wire x1="221.41" y1="30.24" x2="234.315" y2="30.24" width="1.016" layer="16"/>
 <wire x1="234.315" y1="30.24" x2="234.315" y2="30.48" width="1.016" layer="16"/>
 <wire x1="243.97" y1="30.24" x2="236.855" y2="30.24" width="1.016" layer="16"/>
 <wire x1="236.855" y1="30.24" x2="236.855" y2="30.48" width="1.016" layer="16"/>
-<wire x1="134.898165625" y1="30.3784" x2="132.358165625" y2="30.3784" width="0" layer="19" extent="1-1"/>
+<wire x1="121.01" y1="30.24" x2="133.628165625" y2="30.24" width="1.016" layer="16"/>
+<wire x1="133.628165625" y1="30.24" x2="133.628165625" y2="30.3784" width="1.016" layer="16"/>
+<wire x1="143.57" y1="30.24" x2="136.168165625" y2="30.24" width="1.016" layer="16"/>
+<wire x1="136.168165625" y1="30.24" x2="136.168165625" y2="30.3784" width="1.016" layer="16"/>
+<wire x1="136.168165625" y1="30.3784" x2="133.628165625" y2="30.3784" width="0" layer="19" extent="1-1"/>
 <wire x1="236.855" y1="30.48" x2="234.315" y2="30.48" width="0" layer="19" extent="1-1"/>
 </signal>
@@
 <wire x1="171.21" y1="27.7" x2="193.77" y2="27.7" width="1.016" layer="16"/>
 <wire x1="196.31" y1="27.7" x2="218.87" y2="27.7" width="1.016" layer="16"/>
-<wire x1="143.57" y1="27.7" x2="134.898165625" y2="27.7" width="1.016" layer="16"/>
-<wire x1="134.898165625" y1="27.7" x2="134.898165625" y2="27.8384" width="1.016" layer="16"/>
-<wire x1="121.01" y1="27.7" x2="132.358165625" y2="27.7" width="1.016" layer="16"/>
-<wire x1="132.358165625" y1="27.7" x2="132.358165625" y2="27.8384" width="1.016" layer="16"/>
 <wire x1="243.97" y1="27.7" x2="236.855" y2="27.7" width="1.016" layer="16"/>
 <wire x1="236.855" y1="27.7" x2="236.855" y2="27.94" width="1.016" layer="16"/>
 <wire x1="221.41" y1="27.7" x2="234.315" y2="27.7" width="1.016" layer="16"/>
 <wire x1="234.315" y1="27.7" x2="234.315" y2="27.94" width="1.016" layer="16"/>
-<wire x1="134.898165625" y1="27.8384" x2="132.358165625" y2="27.8384" width="0" layer="19" extent="1-1"/>
+<wire x1="143.57" y1="27.7" x2="136.168165625" y2="27.7" width="1.016" layer="16"/>
+<wire x1="136.168165625" y1="27.7" x2="136.168165625" y2="27.8384" width="1.016" layer="16"/>
+<wire x1="121.01" y1="27.7" x2="133.628165625" y2="27.7" width="1.016" layer="16"/>
+<wire x1="133.628165625" y1="27.7" x2="133.628165625" y2="27.8384" width="1.016" layer="16"/>
+<wire x1="136.168165625" y1="27.8384" x2="133.628165625" y2="27.8384" width="0" layer="19" extent="1-1"/>
 <wire x1="236.855" y1="27.94" x2="234.315" y2="27.94" width="0" layer="19" extent="1-1"/>
 </signal>

Commit message: Add files via upload
Parts:
- C1, C10, C11, C2, C4, C5, C7, C8: device rcl:E2,5-6 -> rcl:C025-025X050
- moved LED1 2.54 mm to (374.1, 31.8)
- moved R1 2.54 mm to (369.1, 31.8)
- moved J8 1.78 mm to (361.9, 6.35)
- moved J5 1.78 mm to (361.9, 36.6)
- moved LED2 1.27 mm to (374.1, 11.4)
- moved LED3 1.27 mm to (374.1, 21.6)
- moved R2 1.27 mm to (369.1, 21.6)
- moved R3 1.27 mm to (369.1, 11.4)
- moved J7 0.89 mm to (361.9, 16.1)
- moved J6 0.43 mm to (361.9, 26.3)
Connections:
- net +12V: now also C1.1, C10.1, C4.1, C7.1; no longer C1.+, C10.+, C4.+, C7.+
- net -12V: now also C11.2, C2.2, C5.2, C8.2; no longer C11.-, C2.-, C5.-, C8.-
- net 0V: now also C1.2, C10.2, C11.1, C2.1, C4.2, C5.1, C7.2, C8.1; no longer C1.-, C10.-, C11.+, C2.+, C4.-, C5.+, C7.-, C8.+
Routing:
- net -12V: track 366.8 -> 368.8 mm
- net +5V: track 377.4 -> 378.2 mm
